Commit message: Scaling meshes by 0.001. Scaleing factor in .xacro not to be used

File: soft_hand_description/model/soft_hand.urdf.xacro (robot description, xacro)
@@ -53,4 +53,5 @@
 	<xacro:property name="synergy_damping" value="0.0" />
 	<xacro:property name="synergy_friction" value="0.0" />
+	<xacro:property name="pi" value="3.14159" />
 	<!-- SOFT FINGER model -->
 	<!-- 4 fingers are equal (index, middle, ring, little) -->
@@ -79,11 +80,11 @@
 			<visual>
 				<geometry>
-					<mesh filename="package://soft_hand_description/meshes/knuckle.stl" scale=" .001 .001 .001" />
-				</geometry>
-				<material name="SoftHand/DarkGrey" />
-			</visual>
-			<collision>
-				<geometry>
-					<mesh filename="package://soft_hand_description/meshes/knuckle_collision.stl" scale=" .001 .001 .001" />
+					<mesh filename="package://soft_hand_description/meshes/knuckle.stl" />
+				</geometry>
+				<material name="SoftHand/DarkGrey" />
+			</visual>
+			<collision>
+				<geometry>
+					<mesh filename="package://soft_hand_description/meshes/knuckle_collision.stl" />
 				</geometry>
 			</collision>
@@ -123,11 +124,11 @@
 			<visual>
 				<geometry>
-					<mesh filename="package://soft_hand_description/meshes/phalanx.stl" scale=" .001 .001 .001" />
-				</geometry>
-				<material name="SoftHand/DarkGrey" />
-			</visual>
-			<collision>
-				<geometry>
-					<mesh filename="package://soft_hand_description/meshes/phalanx_collision.stl" scale=" .001 .001 .001" />
+					<mesh filename="package://soft_hand_description/meshes/phalanx.stl" />
+				</geometry>
+				<material name="SoftHand/DarkGrey" />
+			</visual>
+			<collision>
+				<geometry>
+					<mesh filename="package://soft_hand_description/meshes/phalanx_collision.stl" />
 				</geometry>
 			</collision>
@@ -167,11 +168,11 @@
 			<visual>
 				<geometry>
-					<mesh filename="package://soft_hand_description/meshes/phalanx.stl" scale=" .001 .001 .001" />
-				</geometry>
-				<material name="SoftHand/DarkGrey" />
-			</visual>
-			<collision>
-				<geometry>
-					<mesh filename="package://soft_hand_description/meshes/phalanx_collision.stl" scale=" .001 .001 .001" />
+					<mesh filename="package://soft_hand_description/meshes/phalanx.stl" />
+				</geometry>
+				<material name="SoftHand/DarkGrey" />
+			</visual>
+			<collision>
+				<geometry>
+					<mesh filename="package://soft_hand_description/meshes/phalanx_collision.stl" />
 				</geometry>
 			</collision>
@@ -211,11 +212,11 @@
 			<visual>
 				<geometry>
-					<mesh filename="package://soft_hand_description/meshes/fingertip.stl" scale=" .001 .001 .001" />
-				</geometry>
-				<material name="SoftHand/DarkGrey" />
-			</visual>
-			<collision>
-				<geometry>
-					<mesh filename="package://soft_hand_description/meshes/fingertip_collision.stl" scale=" .001 .001 .001" />
+					<mesh filename="package://soft_hand_description/meshes/fingertip.stl" />
+				</geometry>
+				<material name="SoftHand/DarkGrey" />
+			</visual>
+			<collision>
+				<geometry>
+					<mesh filename="package://soft_hand_description/meshes/fingertip_collision.stl" />
 				</geometry>
 			</collision>
@@ -244,5 +245,5 @@
 				<visual>
 					<geometry>
-						<mesh filename="package://soft_hand_description/meshes/thumb_knuckle_left.stl" scale=" .001 .001 .001" />
+						<mesh filename="package://soft_hand_description/meshes/thumb_knuckle_left.stl" />
 					</geometry>
 					<material name="SoftHand/DarkGrey" />
@@ -250,5 +251,5 @@
 				<collision>
 					<geometry>
-						<mesh filename="package://soft_hand_description/meshes/thumb_knuckle_left_collision.stl" scale=" .001 .001 .001" />
+						<mesh filename="package://soft_hand_description/meshes/thumb_knuckle_left_collision.stl" />
 					</geometry>
 				</collision>
@@ -286,5 +287,5 @@
 				<visual>
 					<geometry>
-						<mesh filename="package://soft_hand_description/meshes/thumb_knuckle_right.stl" scale=" .001 .001 .001" />
+						<mesh filename="package://soft_hand_description/meshes/thumb_knuckle_right.stl" />
 					</geometry>
 					<material name="SoftHand/DarkGrey" />
@@ -292,5 +293,5 @@
 				<collision>
 					<geometry>
-						<mesh filename="package://soft_hand_description/meshes/thumb_knuckle_right_collision.stl" scale=" .001 .001 .001" />
+						<mesh filename="package://soft_hand_description/meshes/thumb_knuckle_right_collision.stl" />
 					</geometry>
 				</collision>
@@ -332,11 +333,11 @@
 			<visual>
 				<geometry>
-					<mesh filename="package://soft_hand_description/meshes/phalanx.stl" scale=" .001 .001 .001" />
-				</geometry>
-				<material name="SoftHand/DarkGrey" />
-			</visual>
-			<collision>
-				<geometry>
-					<mesh filename="package://soft_hand_description/meshes/phalanx_collision.stl" scale=" .001 .001 .001" />
+					<mesh filename="package://soft_hand_description/meshes/phalanx.stl" />
+				</geometry>
+				<material name="SoftHand/DarkGrey" />
+			</visual>
+			<collision>
+				<geometry>
+					<mesh filename="package://soft_hand_description/meshes/phalanx_collision.stl" />
 				</geometry>
 			</collision>
@@ -376,11 +377,11 @@
 			<visual>
 				<geometry>
-					<mesh filename="package://soft_hand_description/meshes/fingertip.stl" scale=" .001 .001 .001" />
-				</geometry>
-				<material name="SoftHand/DarkGrey" />
-			</visual>
-			<collision>
-				<geometry>
-					<mesh filename="package://soft_hand_description/meshes/fingertip_collision.stl" scale=" .001 .001 .001" />
+					<mesh filename="package://soft_hand_description/meshes/fingertip.stl" />
+				</geometry>
+				<material name="SoftHand/DarkGrey" />
+			</visual>
+			<collision>
+				<geometry>
+					<mesh filename="package://soft_hand_description/meshes/fingertip_collision.stl" />
 				</geometry>
 			</collision>
@@ -420,5 +421,5 @@
 				<visual>
 					<geometry>
-						<mesh filename="package://soft_hand_description/meshes/palm_left.stl" scale=" .001 .001 .001" />
+						<mesh filename="package://soft_hand_description/meshes/palm_left.stl" />
 					</geometry>
 					<material name="SoftHand/DarkGrey" />
@@ -426,5 +427,5 @@
 				<collision>
 					<geometry>
-						<mesh filename="package://soft_hand_description/meshes/palm_left_collision.stl" scale=" .001 .001 .001" />
+						<mesh filename="package://soft_hand_description/meshes/palm_left_collision.stl" />
 					</geometry>
 				</collision>
@@ -433,5 +434,5 @@
 				<visual>
 					<geometry>
-						<mesh filename="package://soft_hand_description/meshes/palm_right.stl" scale=" .001 .001 .001" />
+						<mesh filename="package://soft_hand_description/meshes/palm_right.stl"/>
 					</geometry>
 					<material name="SoftHand/DarkGrey" />
@@ -439,5 +440,5 @@
 				<collision>
 					<geometry>
-						<mesh filename="package://soft_hand_description/meshes/palm_right_collision.stl" scale=" .001 .001 .001" />
+						<mesh filename="package://soft_hand_description/meshes/palm_right_collision.stl" />
 					</geometry>
 				</collision>
