Commit message: Using fake smaller inertia

File: soft_hand_description/model/soft_hand.inertia.xacro (robot description, xacro)
@@ -12,5 +12,5 @@
     <xacro:property name="gr_to_Kg" value="0.01"/>
     <!-- not so negligible, otherwise simulation fails -->
-    <xacro:property name="negligible_mass" value="${10*gr_to_Kg}"/>
+    <xacro:property name="negligible_mass" value="${1*gr_to_Kg}"/>
     <xacro:property name="negligible_inertia">
         <origin xyz="0 0 0"/>
