Commit message: correcting gripper model

File: soft_hand_description/model/soft_gripper.urdf.xacro (robot description, xacro)
@@ -92,5 +92,5 @@
 		<!-- PROXIMAL PHALANGE -->
 		<joint name="${name}_inner_joint" type="revolute">
-			<origin xyz="0.0 0 0" rpy="0 0 0" />
+			<origin xyz="-0.013 0 0" rpy="0 0 0" />
 			<parent link="${name}_knuckle_link"/>
 			<child link="${name}_fake_link1"/>
@@ -108,5 +108,5 @@
 		</link>
 		<joint name="${name}_inner_joint_mimic" type="revolute">
-			<origin xyz="-0.013 0 0" rpy="0 0 0" />
+			<origin xyz="0.013 0 0" rpy="0 0 0" />
 			<parent link="${name}_fake_link1"/>
 			<child link="${name}_proximal_link"/>
@@ -427,5 +427,5 @@
 				<collision>
 					<geometry>
-						<mesh filename="package://soft_hand_description/meshes/gripper_palm.stl" />
+						<mesh filename="package://soft_hand_description/meshes/gripper_palm_collision.stl" />
 					</geometry>
 				</collision>
@@ -440,5 +440,5 @@
 				<collision>
 					<geometry>
-						<mesh filename="package://soft_hand_description/meshes/gripper_palm.stl" />
+						<mesh filename="package://soft_hand_description/meshes/gripper_palm_collision.stl" />
 					</geometry>
 				</collision>
